File: Centipedes.brd (EAGLE design)
At the start: 20.3 x 109.2 mm, 50 parts, among them IC2 REG1117 5.0V, IC3 MCP6002, IC4 ATMEGA328P-AU, J1 , J15 ICSP, J2 THONKICONNNEW, J3 THONKICONNNEW, J4 THONKICONNNEW, J5 THONKICONNNEW, Q1 20MHZ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

Commit message: Add files via upload
Parts:
- added C8: 22uf, rcl:PANASONIC_C
Connections:
- net GND: now also C8.+
- net VEE: now also C8.-
Routing:
- net VEE: track 75.7 -> 81.2 mm
Changed lines of the file:
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@@
 <drawing>
 <settings>
-<setting alwaysvectorfont="no"/>
+<setting alwaysvectorfont="yes"/>
 <setting verticaltext="up"/>
 </settings>
-<grid distance="0.001" unitdist="inch" unit="inch" style="dots" multiple="1" display="yes" altdistance="5" altunitdist="mil" altunit="mil"/>
+<grid distance="0.01" unitdist="inch" unit="inch" style="dots" multiple="1" display="yes" altdistance="5" altunitdist="mil" altunit="mil"/>
 <layers>
 <layer number="1" name="Top" color="4" fill="1" visible="yes" active="yes"/>
@@
 <wire x1="20.371" y1="109.21" x2="0.0635" y2="109.21" width="0" layer="20"/>
 <wire x1="0.0635" y1="109.21" x2="0.0635" y2="0" width="0" layer="20"/>
-<text x="19.558" y="108.712" size="1.778" layer="26" rot="MR270">CENTIPEDES</text>
-<text x="2.032" y="108.712" size="1.27" layer="26" rot="SMR270">HOLMES MODULAR</text>
+<text x="19.05" y="108.204" size="0.889" layer="26" rot="MR270">CENTIPEDES</text>
+<text x="1.016" y="97.282" size="0.889" layer="26" rot="SMR90">HOLMES MODULAR</text>
 <text x="19.812" y="90.678" size="1.27" layer="26" rot="SMR0">C.J.H.</text>
 <wire x1="20.32" y1="109.22" x2="17.018" y2="109.22" width="0.1524" layer="26"/>
-<wire x1="17.018" y1="109.22" x2="17.018" y2="92.456" width="0.1524" layer="26"/>
-<wire x1="17.018" y1="92.456" x2="20.32" y2="92.456" width="0.1524" layer="26"/>
-<wire x1="20.32" y1="92.456" x2="20.32" y2="109.22" width="0.1524" layer="26"/>
-<wire x1="0" y1="109.22" x2="0" y2="91.186" width="0.1524" layer="26"/>
-<wire x1="0" y1="91.186" x2="3.048" y2="91.186" width="0.1524" layer="26"/>
-<wire x1="3.048" y1="91.186" x2="3.048" y2="109.22" width="0.1524" layer="26"/>
+<wire x1="17.018" y1="109.22" x2="17.018" y2="99.822" width="0.1524" layer="26"/>
+<wire x1="17.018" y1="99.822" x2="20.32" y2="99.822" width="0.1524" layer="26"/>
+<wire x1="20.32" y1="99.822" x2="20.32" y2="109.22" width="0.1524" layer="26"/>
+<wire x1="0" y1="109.22" x2="0" y2="96.012" width="0.1524" layer="26"/>
+<wire x1="0" y1="96.012" x2="3.048" y2="96.012" width="0.1524" layer="26"/>
+<wire x1="3.048" y1="96.012" x2="3.048" y2="109.22" width="0.1524" layer="26"/>
 <text x="19.812" y="87.63" size="1.27" layer="26" rot="MR0">v2</text>
 <text x="12.0904" y="40.132" size="1.778" layer="26" rot="MR0">.</text>
@@
 <attribute name="VALUE" x="10.414" y="62.357" size="1.27" layer="27" rot="R270"/>
 </element>
+<element name="C8" library="rcl" library_urn="urn:adsk.eagle:library:334" package="PANASONIC_C" package3d_urn="urn:adsk.eagle:package:23422/2" value="22uf" x="3.6068" y="91.9988" smashed="yes" rot="MR270">
+<attribute name="NAME" x="0.8568" y="94.5988" size="1.016" layer="26" rot="MR270"/>
+<attribute name="POPULARITY" value="5" x="3.6068" y="91.9988" size="1.778" layer="28" rot="MR270" display="off"/>
+<attribute name="SPICEPREFIX" value="C" x="3.6068" y="91.9988" size="1.778" layer="28" rot="MR270" display="off"/>
+<attribute name="VALUE" x="7.3818" y="94.6488" size="1.016" layer="28" rot="MR270"/>
+</element>
 </elements>
 <signals>
@@
 <wire x1="1.524" y1="56.769" x2="1.524" y2="49.9364" width="0.508" layer="1"/>
 <wire x1="1.7272" y1="49.7332" x2="1.524" y2="49.9364" width="0.508" layer="1"/>
-<wire x1="1.7158" y1="56.3232" x2="1.7018" y2="56.3232" width="0.508" layer="16"/>
-<wire x1="1.651" y1="56.374" x2="1.7018" y2="56.3232" width="0.508" layer="16"/>
+<wire x1="1.651" y1="56.374" x2="1.4478" y2="56.5772" width="0.508" layer="16"/>
 <wire x1="3.5814" y1="55.518" x2="2.4956" y2="55.518" width="0.508" layer="16"/>
 <wire x1="1.651" y1="56.3626" x2="1.651" y2="56.374" width="0.508" layer="16"/>
@@
 <via x="2.286" y="2.286" extent="1-16" drill="0.35"/>
 <via x="9.906" y="19.812" extent="1-16" drill="0.35"/>
+<contactref element="C8" pad="+"/>
 </signal>
 <signal name="+5V">
@@
 </signal>
 <signal name="VEE">
-<contactref element="D1" pad="-"/>
 <contactref element="R1" pad="2"/>
 <wire x1="9.906" y1="27.7368" x2="9.906" y2="27.725" width="0.1524" layer="16"/>
 <via x="11.2776" y="28.3464" extent="1-16" drill="0.35"/>
 <via x="10.0584" y="92.202" extent="1-16" drill="0.35" diameter="0.95" shape="octagon"/>
-<wire x1="8.86" y1="93.47" x2="10.0584" y2="92.2716" width="1.016" layer="16"/>
 <wire x1="10.0584" y1="92.2716" x2="10.0584" y2="92.202" width="1.016" layer="16"/>
 <wire x1="10.0584" y1="92.202" x2="10.112" y2="92.1484" width="1.016" layer="1"/>
@@
 <wire x1="11.2776" y1="28.3464" x2="10.668" y2="27.7368" width="0.8128" layer="16"/>
 <wire x1="10.668" y1="27.7368" x2="9.906" y2="27.7368" width="0.8128" layer="16"/>
+<contactref element="D1" pad="-"/>
+<contactref element="C8" pad="-"/>
+<wire x1="8.86" y1="93.47" x2="4.1856" y2="93.47" width="1.016" layer="16"/>
+<wire x1="4.1856" y1="93.47" x2="3.6068" y2="94.0488" width="1.016" layer="16"/>
+<wire x1="8.86" y1="93.47" x2="10.0584" y2="92.2716" width="1.016" layer="16"/>
 </signal>
 <signal name="REF-5V">
